Commit message: initial - Ian departure

File: config/platform.urdf (robot description, URDF)
Before this commit: robot vehicle_platform, 8 links, 7 joints
Links:
- removed link mobileye
- removed link radar_fl
- removed link radar_fr
- removed link radar_rl
- removed link radar_rr
- added link imu
Joints:
- removed joint mobileye
- removed joint radar_fl
- removed joint radar_fr
- removed joint radar_rl
- removed joint radar_rr
- added joint imu: type fixed, parent base_link, child imu, origin xyz=0 0 0 rpy=0 0 0
- joint lidar: origin xyz=1.02 0 2.23 rpy=0 0 0 -> xyz=1.02 0 1.78734 rpy=0 0 0
- joint radar_fc: origin xyz=4 0 0.57 rpy=0 0 0 -> xyz=4 0 0.07 rpy=0 0 0

Commit message: LiDAR yaw offset

File: config/platform.urdf (robot description, URDF)
Before this commit: robot vehicle_platform, 4 links, 3 joints
Joints:
- joint lidar: origin xyz=1.02 0 1.78734 rpy=0 0 0 -> xyz=1.02 0 1.78734 rpy=0 0 0.015

Commit message: corrected lidar tf

File: config/platform.urdf (robot description, URDF)
Before this commit: robot vehicle_platform, 4 links, 3 joints
Joints:
- joint lidar: origin xyz=1.02 0 1.78734 rpy=0 0 0.015 -> xyz=1.02 0 1.78734 rpy=0 0 -0.021

Commit message: added decond lidar config

File: config/platform.urdf (robot description, URDF)
Before this commit: robot vehicle_platform, 4 links, 3 joints
Links:
- added link lidar_front
Joints:
- added joint lidar_front: type fixed, parent base_link, child lidar_front, origin xyz=1.98 0 1.3753 rpy=0 0.15 -0.021

Commit message: corrected tf lidar center + front

File: config/platform.urdf (robot description, URDF)
Before this commit: robot vehicle_platform, 5 links, 4 joints
Joints:
- joint lidar: origin xyz=1.02 0 1.78734 rpy=0 0 -0.021 -> xyz=1.02 0 1.78734 rpy=0 0 0.017
- joint lidar_front: origin xyz=1.98 0 1.3753 rpy=0 0.15 -0.021 -> xyz=1.97 0 1.3753 rpy=-0.011 0.204 -0.037

Commit message: lidar front tf (good?)

File: config/platform.urdf (robot description, URDF)
Before this commit: robot vehicle_platform, 5 links, 4 joints
Joints:
- joint lidar_front: origin xyz=1.97 0 1.3753 rpy=-0.011 0.204 -0.037 -> xyz=1.97 0 1.3163 rpy=-0.008 0.197 -0.037

Commit message: fixed ip for velodyne + tf fixes for ouster

File: config/platform.urdf (robot description, URDF)
Before this commit: robot vehicle_platform, 5 links, 4 joints
Links:
- removed link lidar
- added link lidar_center/os_sensor
Joints:
- removed joint lidar
- added joint lidar_center/os_sensor: type fixed, parent base_link, child lidar_center/os_sensor, origin xyz=1.02 0 1.78734 rpy=0 0 0.017

Commit message: ouster driver sync + ext calib

File: config/platform.urdf (robot description, URDF)
Before this commit: robot vehicle_platform, 5 links, 4 joints
Joints:
- joint lidar_center/os_sensor: origin xyz=1.02 0 1.78734 rpy=0 0 0.017 -> xyz=1.02 0 1.78734 rpy=0 0 0.022
- joint lidar_front: origin xyz=1.97 0 1.3163 rpy=-0.008 0.197 -0.037 -> xyz=1.97 0 1.3163 rpy=0.009 0.193 0.033

Commit message: updated front lidar tf

File: config/platform.urdf (robot description, URDF)
Before this commit: robot vehicle_platform, 5 links, 4 joints
Joints:
- joint lidar_center/os_sensor: origin xyz=1.02 0 1.78734 rpy=0 0 0.022 -> xyz=1.886 -0.033 1.640 rpy=-0.025, 0.237, 0.021
- joint lidar_front: origin xyz=1.97 0 1.3163 rpy=0.009 0.193 0.033 -> xyz=1.92 -0.072 1.639 rpy=-0.004 0.242 0.124

Commit message: more conf for ouster

File: config/platform.urdf (robot description, URDF)
Before this commit: robot vehicle_platform, 5 links, 4 joints
Joints:
- joint lidar_center/os_sensor: origin xyz=1.886 -0.033 1.640 rpy=-0.025, 0.237, 0.021 -> xyz=1.886 -0.033 1.640 rpy=0 0 0.022

Commit message: compatibility for ouster driver + new velodyne driver

File: config/platform.urdf (robot description, URDF)
Before this commit: robot vehicle_platform, 5 links, 4 joints
Links:
- added link lidar
Joints:
- added joint lidar: type fixed, parent lidar_center/os_sensor, child lidar, origin xyz=0 0 0 rpy=0 0 0

Commit message: tf corrections

File: config/platform.urdf (robot description, URDF)
Before this commit: robot vehicle_platform, 6 links, 5 joints
Joints:
- joint lidar_center/os_sensor: origin xyz=1.886 -0.033 1.640 rpy=0 0 0.022 -> xyz=1.02 0 1.78734 rpy=0 0 0.022
- joint lidar_front: origin xyz=1.92 -0.072 1.639 rpy=-0.004 0.242 0.124 -> xyz=1.92 -0.072 1.439 rpy=0.001 0.192 0.028

Commit message: new tf for new ouster lidar

File: config/platform.urdf (robot description, URDF)
Before this commit: robot vehicle_platform, 6 links, 5 joints
Joints:
- joint lidar_center/os_sensor: origin xyz=1.02 0 1.78734 rpy=0 0 0.022 -> xyz=1.02 0 1.78734 rpy=0 0 0.015

Commit message: added nvidia cameras extrinsics to platform urdf

File: config/platform.urdf (robot description, URDF)
Before this commit: robot vehicle_platform, 6 links, 5 joints
Links:
- added link interfacea_link0
- added link interfacea_link1
- added link interfacea_link2
- added link interfacea_link3
Joints:
- added joint interfacea_link0: type fixed, parent lidar, child interfacea_link0, origin xyz=0.777 0.556 -0.475 rpy=-1.569 0.056 -1.148
- added joint interfacea_link1: type fixed, parent lidar, child interfacea_link1, origin xyz=0.848 -0.580 -0.503 rpy=-1.539 -0.021 -2.128
- added joint interfacea_link2: type fixed, parent lidar, child interfacea_link2, origin xyz=0.776 -0.111 -0.457 rpy=-1.584 0.036 -1.604
- added joint interfacea_link3: type fixed, parent lidar, child interfacea_link3, origin xyz=0.858 0.181 -0.486 rpy=-1.572 0.017 -1.613

Commit message: added uncompression + rectification to nvidia cameras launchfile

File: config/platform.urdf (robot description, URDF)
Before this commit: robot vehicle_platform, 10 links, 9 joints
Joints:
- joint interfacea_link0: origin xyz=0.777 0.556 -0.475 rpy=-1.569 0.056 -1.148 -> xyz=0.777 0.556 -0.475 rpy=-1.564 0.052 -1.137
- joint interfacea_link1: origin xyz=0.848 -0.580 -0.503 rpy=-1.539 -0.021 -2.128 -> xyz=0.848 -0.580 -0.503 rpy=-1.529 -0.021 -2.13

Commit message: camera tf now published by driver

File: config/platform.urdf (robot description, URDF)
Before this commit: robot vehicle_platform, 10 links, 9 joints
Links:
- added link camera_fl
- added link camera_fr
Joints:
- added joint camera_fl: type fixed, parent lidar, child camera_fl, origin xyz=1.11787 0.17502 -0.66163 rpy=-1.47631 -0.00633 -1.66711
- added joint camera_fr: type fixed, parent lidar, child camera_fr, origin xyz=1.0776 -0.26893 -0.65117 rpy=-1.40999 0.0939 -2.02844

Commit message: tuned nvidia camera facing forward

File: config/platform.urdf (robot description, URDF)
Before this commit: robot vehicle_platform, 10 links, 9 joints
Joints:
- joint interfacea_link0: origin xyz=0.777 0.556 -0.475 rpy=-1.564 0.052 -1.137 -> xyz=0.777 0.556 -0.475 rpy=-1.594 0.032 -1.477
- joint interfacea_link1: origin xyz=0.848 -0.580 -0.503 rpy=-1.529 -0.021 -2.13 -> xyz=0.848 -0.580 -0.503 rpy=-1.564 0.039 -1.58

Commit message: Added ground_zero transform for testing ground removal

File: config/platform.urdf (robot description, URDF)
Before this commit: robot vehicle_platform, 12 links, 11 joints
Links:
- added link ground_zero
Joints:
- added joint ground_zero: type fixed, parent base_link, child ground_zero, origin xyz=0 0 -0.3 rpy=0 0 0.015

Commit message: Removed rotation from ground_zero tf

File: config/platform.urdf (robot description, URDF)
Before this commit: robot vehicle_platform, 13 links, 12 joints
Joints:
- joint ground_zero: origin xyz=0 0 -0.3 rpy=0 0 0.015 -> xyz=0 0 -0.3 rpy=0 0 0

Commit message: [#11] Added latest velodyne to ouster lidar calibration in urdf

File: config/platform.urdf (robot description, URDF)
Before this commit: robot vehicle_platform, 13 links, 12 joints
Joints:
- joint lidar_front: origin xyz=1.92 -0.072 1.439 rpy=0.001 0.192 0.028 -> xyz= 0.82727 -0.00144 -0.20905 rpy=0.00302 -0.00092 0.0413; parent base_link -> lidar

Commit message: [#374] intrinsics and extrinsic parameter update following lens replacement

File: config/platform.urdf (robot description, URDF)
Before this commit: robot vehicle_platform, 13 links, 12 joints
Joints:
- joint camera_fl: origin xyz=1.11787 0.17502 -0.66163 rpy=-1.47631 -0.00633 -1.66711 -> xyz=1.11787 0.17502 -0.66163 rpy=-1.43531 -0.00833 -1.67511
- joint camera_fr: origin xyz=1.0776 -0.26893 -0.65117 rpy=-1.40999 0.0939 -2.02844 -> xyz=1.0 -0.21 -0.65 rpy=-1.38629 0.01096 -1.8499

Commit message: update extrinsics using leveller

File: config/platform.urdf (robot description, URDF)
Before this commit: robot vehicle_platform, 13 links, 12 joints
Joints:
- joint camera_fl: origin xyz=1.11787 0.17502 -0.66163 rpy=-1.43531 -0.00833 -1.67511 -> xyz=1.11787 0.17502 -0.66163 rpy=-1.44031 -0.04533 -1.67511
- joint camera_fr: origin xyz=1.0 -0.21 -0.65 rpy=-1.38629 0.01096 -1.8499 -> xyz=1.0 -0.21 -0.65 rpy=-1.38629 -0.00604 -1.8549

Commit message: new base to velodyne calibration

File: config/platform.urdf (robot description, URDF)
Before this commit: robot vehicle_platform, 13 links, 12 joints
Links:
- removed link lidar_center/os_sensor
- removed link lidar_front
- added link lidar_center
- added link lidar_front/os_sensor
Joints:
- removed joint lidar_center/os_sensor
- removed joint lidar_front
- added joint lidar_center: type fixed, parent base_link, child lidar_center, origin xyz=1.02 0 1.78734 rpy=0 0 -0.0459
- added joint lidar_front/os_sensor: type fixed, parent lidar, child lidar_front/os_sensor, origin xyz= 0.82727 -0.00144 -0.20905 rpy=0.00302 -0.00092 0.0413
- joint lidar: parent lidar_center/os_sensor -> lidar_center

Commit message: updating calibration parameters with wrong camera_fr

File: config/platform.urdf (robot description, URDF)
Before this commit: robot vehicle_platform, 13 links, 12 joints
Joints:
- joint camera_fl: origin xyz=1.11787 0.17502 -0.66163 rpy=-1.44031 -0.04533 -1.67511 -> xyz=0.187 0.23 -0.34 rpy=-1.40831 -0.01033 -1.68511; parent lidar -> lidar_front/os_sensor
- joint camera_fr: origin xyz=1.0 -0.21 -0.65 rpy=-1.38629 -0.00604 -1.8549 -> xyz=-1.87 -0.23 -0.33 rpy=-1.30929 -0.01504 -1.8479; parent lidar -> lidar_front/os_sensor
- joint lidar_front/os_sensor: origin xyz= 0.82727 -0.00144 -0.20905 rpy=0.00302 -0.00092 0.0413 -> xyz= 0.90509 0.03386 -0.344505 rpy=0.0167 0.05216 0.06163

Commit message: updating nvidia cameras extrinsics

File: config/platform.urdf (robot description, URDF)
Before this commit: robot vehicle_platform, 13 links, 12 joints
Joints:
- joint interfacea_link0: origin xyz=0.777 0.556 -0.475 rpy=-1.594 0.032 -1.477 -> xyz=-0.055 0.57 -0.125 rpy=-1.536 0.014 -1.535; parent lidar -> lidar_front/os_sensor
- joint interfacea_link1: origin xyz=0.848 -0.580 -0.503 rpy=-1.564 0.039 -1.58 -> xyz=-0.055 -0.54 -0.125 rpy=-1.508 -0.013 -1.565; parent lidar -> lidar_front/os_sensor
- joint interfacea_link2: origin xyz=0.776 -0.111 -0.457 rpy=-1.584 0.036 -1.604 -> xyz=-0.01 -0.14 -0.125 rpy=-1.532 0.004 -1.599; parent lidar -> lidar_front/os_sensor
- joint interfacea_link3: origin xyz=0.858 0.181 -0.486 rpy=-1.572 0.017 -1.613 -> xyz=-0.015 0.17 -0.125 rpy=-1.527 -0.007 -1.597; parent lidar -> lidar_front/os_sensor

Commit message: update platform.urdf with calibs. Remove diagnostic errors after confi change

File: config/platform.urdf (robot description, URDF)
Before this commit: robot vehicle_platform, 13 links, 12 joints
Joints:
- joint camera_fr: origin xyz=-1.87 -0.23 -0.33 rpy=-1.30929 -0.01504 -1.8479 -> xyz=0.23 -0.227 -0.33 rpy=-1.30929 -0.02004 -1.8479
- joint interfacea_link0: origin xyz=-0.055 0.57 -0.125 rpy=-1.536 0.014 -1.535 -> xyz=-0.08 0.57 -0.125 rpy=-1.544 0.008 -1.534
- joint interfacea_link1: origin xyz=-0.055 -0.54 -0.125 rpy=-1.508 -0.013 -1.565 -> xyz=-0.104 -0.54 -0.125 rpy=-1.508 -0.018 -1.564
- joint interfacea_link2: origin xyz=-0.01 -0.14 -0.125 rpy=-1.532 0.004 -1.599 -> xyz=-0.018 -0.14 -0.125 rpy=-1.532 0.004 -1.606
- joint interfacea_link3: origin xyz=-0.015 0.17 -0.125 rpy=-1.527 -0.007 -1.597 -> xyz=-0.018 0.17 -0.125 rpy=-1.524 -0.003 -1.599

Commit message: changing cam calibration and calibration launch/rviz file

File: config/platform.urdf (robot description, URDF)
Before this commit: robot vehicle_platform, 13 links, 12 joints
Joints:
- joint camera_fl: origin xyz=0.187 0.23 -0.34 rpy=-1.40831 -0.01033 -1.68511 -> xyz=1.059 0.279 -0.689 rpy=-1.41203 -0.01469 -1.41365; parent lidar_front/os_sensor -> lidar_center
- joint camera_fr: origin xyz=0.23 -0.227 -0.33 rpy=-1.30929 -0.02004 -1.8479 -> xyz=1.130 -0.174 -0.689 rpy=-1.36404 -0.00223 -1.78766; parent lidar_front/os_sensor -> lidar_center

Commit message: update ouster calib after changing pose.

File: config/platform.urdf (robot description, URDF)
Before this commit: robot vehicle_platform, 13 links, 12 joints
Joints:
- joint lidar_front/os_sensor: origin xyz= 0.90509 0.03386 -0.344505 rpy=0.0167 0.05216 0.06163 -> xyz=[0.85079 0.0400148 -0.340915 rpy=-0.0 0.0 0.858853

Commit message: fixed typo in platform.urdf

File: config/platform.urdf (robot description, URDF)
Before this commit: robot vehicle_platform, 13 links, 12 joints
Joints:
- joint lidar_front/os_sensor: origin xyz=[0.85079 0.0400148 -0.340915 rpy=-0.0 0.0 0.858853 -> xyz=0.85079 0.0400148 -0.340915 rpy=-0.0 0.0 0.858853

Commit message: tuning the lidar-lidar and lidar-cam calibration

File: config/platform.urdf (robot description, URDF)
Before this commit: robot vehicle_platform, 13 links, 12 joints
Joints:
- joint camera_fl: origin xyz=1.059 0.279 -0.689 rpy=-1.41203 -0.01469 -1.41365 -> xyz=1.009 0.278 -0.689 rpy=-1.40103 -0.00669 -1.41965
- joint lidar_front/os_sensor: origin xyz=0.85079 0.0400148 -0.340915 rpy=-0.0 0.0 0.858853 -> xyz=0.84979 0.06501 -0.28092 rpy=0.0119 0.003 0.86855; parent lidar -> lidar_center

Commit message: updating nvidia cameras calibration

File: config/platform.urdf (robot description, URDF)
Before this commit: robot vehicle_platform, 13 links, 12 joints
Joints:
- joint interfacea_link0: origin xyz=-0.08 0.57 -0.125 rpy=-1.544 0.008 -1.534 -> xyz=0.8225 0.5925 -0.412 rpy=-1.594 0.042 -1.4638; parent lidar_front/os_sensor -> lidar_center
- joint interfacea_link1: origin xyz=-0.104 -0.54 -0.125 rpy=-1.508 -0.018 -1.564 -> xyz=0.8776 -0.5095 -0.412 rpy=-1.564 0.008 -1.52; parent lidar_front/os_sensor -> lidar_center
- joint interfacea_link2: origin xyz=-0.018 -0.14 -0.125 rpy=-1.532 0.004 -1.606 -> xyz=0.91965 -0.1074 -0.412 rpy=-1.602 0.022 -1.544; parent lidar_front/os_sensor -> lidar_center
- joint interfacea_link3: origin xyz=-0.018 0.17 -0.125 rpy=-1.524 -0.003 -1.599 -> xyz=0.9045 0.1956 -0.412 rpy=-1.589 -0.003 -1.533; parent lidar_front/os_sensor -> lidar_center

Commit message: Updated Nvidia link3 extrinsics orientation and position values in platform.urdf

File: config/platform.urdf (robot description, URDF)
Before this commit: robot vehicle_platform, 13 links, 12 joints
Joints:
- joint interfacea_link3: origin xyz=0.9045 0.1956 -0.412 rpy=-1.589 -0.003 -1.533 -> xyz=0.6500 0.1600 -0.4800 rpy=-1.550 0.017 -1.568

Commit message: Changed nv link3 position and orientation back to previous values

File: config/platform.urdf (robot description, URDF)
Before this commit: robot vehicle_platform, 13 links, 12 joints
Joints:
- joint interfacea_link3: origin xyz=0.6500 0.1600 -0.4800 rpy=-1.550 0.017 -1.568 -> xyz=0.9045 0.1956 -0.4120 rpy=-1.589 -0.003 -1.533

Commit message: [#484] removed ground_zero from platform.urdf, replaced with base_footprint

File: config/platform.urdf (robot description, URDF)
Before this commit: robot vehicle_platform, 14 links, 13 joints
Links:
- removed link ground_zero
Joints:
- removed joint ground_zero

Commit message: extrinsic calibration, link_0_1 done at delta (need improvement), link_2_3 erm

File: config/platform.urdf (robot description, URDF)
Before this commit: robot vehicle_platform, 13 links, 12 joints
Joints:
- joint interfacea_link0: origin xyz=0.68 0.703 -0.511 rpy=-1.5899949 0.0357792 -1.476199 -> xyz=0.514 0.404 -0.472 rpy=-1.572367 0.051313 -0.704764
- joint interfacea_link1: origin xyz=0.73 -0.304 -0.48 rpy=-1.624552 0.01867502 -1.8217746 -> xyz=0.759 -0.336 -0.530 rpy=-1.631359 -0.029321 -2.525666
- joint interfacea_link2: origin xyz=0.896 0.036 -0.513 rpy=-1.588773 0.03054326 -1.5613715 -> xyz=0.987 0.036 -0.570 rpy=-1.601863 0.033859 -1.533795
- joint interfacea_link3: origin xyz=1.008 0.284 -0.507 rpy=-1.579348 0.017104226 -1.54950330 -> xyz=0.954 0.142 -0.502 rpy=-1.589122 0.014137 -1.541823

Commit message: [#479] updated extrinsics for nvida cameras

File: config/platform.urdf (robot description, URDF)
Before this commit: robot vehicle_platform, 13 links, 12 joints
Joints:
- joint interfacea_link0: origin xyz=0.514 0.404 -0.472 rpy=-1.572367 0.051313 -0.704764 -> xyz=0.77 0.62 -0.49 rpy=-1.576381 0.001396 -0.182561
- joint interfacea_link1: origin xyz=0.759 -0.336 -0.530 rpy=-1.631359 -0.029321 -2.525666 -> xyz=0.83 -0.51 -0.49 rpy=-1.63537 0.001919 -2.844538
- joint interfacea_link2: origin xyz=0.987 0.036 -0.570 rpy=-1.601863 0.033859 -1.533795 -> xyz=0.89 0.04 -0.49 rpy=-1.601863 0.033684 -1.533795
- joint interfacea_link3: origin xyz=0.954 0.142 -0.502 rpy=-1.589122 0.014137 -1.541823 -> xyz=0.89 0.09 -0.49 rpy=-1.58912 0.024434 -1.533097

Commit message: Release 0.1

File: config/platform.urdf (robot description, URDF)
Before this commit: robot vehicle_platform, 8 links, 7 joints
Links:
- removed link mobileye
- removed link radar_fl
- removed link radar_fr
- removed link radar_rl
- removed link radar_rr
- added link base_footprint
- added link camera_fl
- added link camera_fr
- added link imu
- added link interfacea_link0
- added link interfacea_link1
- added link interfacea_link2
- added link interfacea_link3
- added link lidar_center
- added link lidar_front/os_sensor
Joints:
- removed joint mobileye
- removed joint radar_fl
- removed joint radar_fr
- removed joint radar_rl
- removed joint radar_rr
- added joint base_footprint: type fixed, parent base_link, child base_footprint, origin xyz=0 0 -0.6 rpy=0 0 0
- added joint camera_fl: type fixed, parent lidar_center, child camera_fl, origin xyz=1.131 0.338 -0.747 rpy=-1.4044664 -0.00261799 -1.422443
- added joint camera_fr: type fixed, parent lidar_center, child camera_fr, origin xyz=1.152 -0.168 -0.747 rpy=-1.378984 0.04415683 -1.7793631
- added joint imu: type fixed, parent base_link, child imu, origin xyz=0 0 0 rpy=0 0 0
- added joint interfacea_link0: type fixed, parent lidar_center, child interfacea_link0, origin xyz=0.77 0.62 -0.49 rpy=-1.576381 0.001396 -0.182561
- added joint interfacea_link1: type fixed, parent lidar_center, child interfacea_link1, origin xyz=0.83 -0.51 -0.49 rpy=-1.63537 0.001919 -2.844538
- added joint interfacea_link2: type fixed, parent lidar_center, child interfacea_link2, origin xyz=0.89 0.04 -0.49 rpy=-1.601863 0.033684 -1.533795
- added joint interfacea_link3: type fixed, parent lidar_center, child interfacea_link3, origin xyz=0.89 0.09 -0.49 rpy=-1.58912 0.024434 -1.533097
- added joint lidar_center: type fixed, parent base_link, child lidar_center, origin xyz=1.02 0 1.51 rpy=-0.02879793 0.0003490659 -0.0459
- added joint lidar_front/os_sensor: type fixed, parent lidar_center, child lidar_front/os_sensor, origin xyz=0.8559 0.0642 -0.4051 rpy=0.003995038 -0.009182 0.8641542
- joint lidar: origin xyz=1.02 0 2.23 rpy=0 0 0 -> xyz=0 0 0 rpy=0 0 0; parent base_link -> lidar_center
- joint radar_fc: origin xyz=4 0 0.57 rpy=0 0 0 -> xyz=4 0 -0.12 rpy=0 0 0

Commit message: Added dummy lidar_0 frame for compatibility with Vella

File: config/platform.urdf (robot description, URDF)
Before this commit: robot vehicle_platform, 13 links, 12 joints
Links:
- added link lidar_0
Joints:
- added joint lidar_0: type fixed, parent lidar_center, child lidar_0, origin xyz=0 0 0 rpy=0 0 0

Commit message: finetuned lidar_center base_link transform yaw angle

File: config/platform.urdf (robot description, URDF)
Before this commit: robot vehicle_platform, 14 links, 13 joints
Joints:
- joint lidar_center: origin xyz=1.02 0 1.51 rpy=-0.02879793 0.0003490659 -0.0459 -> xyz=1.02 0 1.51 rpy=-0.02879793 0.0003490659 -0.055
