Commit message: [#484] base_footprint added and base_link lidar_center transform change

File: config/lexus_model.urdf (robot description, URDF)
Before this commit: robot lexus, 2 links, 1 joints
Joints:
- joint link_BaseLink: origin xyz=0 0 -0.30 rpy=0 0 1.5708 -> xyz=-0.05 0 -0.60 rpy=0 0 1.5708

File: config/platform.urdf (robot description, URDF)
Before this commit: robot vehicle_platform, 13 links, 12 joints
Links:
- added link base_footprint
Joints:
- added joint base_footprint: type fixed, parent base_link, child base_footprint, origin xyz=0 0 -0.6 rpy=0 0 0
- joint camera_fl: origin xyz=1.009 0.278 -0.689 rpy=-1.40103 -0.00669 -1.41965 -> xyz=1.131 0.338 -0.747 rpy=-1.4044664 -0.00261799 -1.422443
- joint camera_fr: origin xyz=1.130 -0.174 -0.689 rpy=-1.36404 -0.00223 -1.78766 -> xyz=1.152 -0.168 -0.747 rpy=-1.378984 0.04415683 -1.7793631
- joint ground_zero: origin xyz=0 0 -0.3 rpy=0 0 0 -> xyz=0 0 -0.6 rpy=0 0 0
- joint interfacea_link0: origin xyz=0.8225 0.5925 -0.412 rpy=-1.594 0.042 -1.4638 -> xyz=0.68 0.703 -0.511 rpy=-1.5899949 0.0357792 -1.476199
- joint interfacea_link1: origin xyz=0.8776 -0.5095 -0.412 rpy=-1.564 0.008 -1.52 -> xyz=0.73 -0.304 -0.48 rpy=-1.624552 0.01867502 -1.8217746
- joint interfacea_link2: origin xyz=0.91965 -0.1074 -0.412 rpy=-1.602 0.022 -1.544 -> xyz=0.896 0.036 -0.513 rpy=-1.588773 0.03054326 -1.5613715
- joint interfacea_link3: origin xyz=0.9045 0.1956 -0.4120 rpy=-1.589 -0.003 -1.533 -> xyz=1.008 0.284 -0.507 rpy=-1.579348 0.017104226 -1.54950330
- joint lidar_center: origin xyz=1.02 0 1.78734 rpy=0 0 -0.0459 -> xyz=1.02 0 1.51 rpy=-0.02879793 0.0003490659 -0.0459
- joint lidar_front/os_sensor: origin xyz=0.84979 0.06501 -0.28092 rpy=0.0119 0.003 0.86855 -> xyz=0.8559 0.0642 -0.4051 rpy=0.003995038 -0.009182 0.8641542
- joint radar_fc: origin xyz=4 0 0.07 rpy=0 0 0 -> xyz=4 0 -0.12 rpy=0 0 0

Commit message: Updated lexus_model transforms, so that it is placed at base_link

File: config/lexus_model.urdf (robot description, URDF)
Before this commit: robot lexus, 2 links, 1 joints
Links:
- link lexus_model: mass 0.001 -> None
Joints:
- removed joint link_BaseLink
- added joint joint_lexus_model: type fixed, parent base_link, child lexus_model, origin xyz=0 0 0 rpy=0 0 0
